Commit message: rviz

File: urdf/robot_model_gazebo.xacro (robot description, xacro)
@@ -7,19 +7,19 @@
 	<!-- KINECT ATTACHMENT -->
 	<xacro:include filename="$(find robot_model_gazebo)/urdf/sensors/kinect.xacro"/>
-	<kinect_sensor parent="kinect_base_link">
+	<xacro:kinect_sensor parent="head_pan_link">
 		<!--origin xyz="0 0 0" rpy="0 0 0" /-->
-	</kinect_sensor>
+	</xacro:kinect_sensor>
 	<!-- LASER ATTACHMENT -->
 	<xacro:include filename="$(find robot_model_gazebo)/urdf/sensors/hokuyo.xacro"/>
-	<hokuyo_sensor parent="upper_base_link">
+	<xacro:hokuyo_sensor parent="upper_base_link">
 		<!--origin xyz="0 0 0" rpy="0 0 0" /-->
-	</hokuyo_sensor>
+	</xacro:hokuyo_sensor>
 	<!-- Import all Gazebo-customization elements, including Gazebo colors, sensors, controller -->
   	<xacro:include filename="$(find robot_model_gazebo)/urdf/robot_model_gazebo.gazebo" />
 	<!-- Add view camera - working -->
 	<xacro:include filename="$(find robot_model_gazebo)/urdf/sensors/view_camera.xacro" />
-	<view_camera_sensor parent="kinect_base_link">
+	<xacro:view_camera_sensor parent="head_pan_link">
 		<!--origin xyz="0 0 0" rpy="0 0 0" /-->
-	</view_camera_sensor>
+	</xacro:view_camera_sensor>
 	<xacro:property name="length_wheel" value="0.075" />
 	<xacro:property name="radius_wheel" value="0.0775" />
@@ -71,5 +71,5 @@
 	</gazebo>
 	<joint name="base_footprint_joint" type="fixed">
-		<origin xyz="0 0 0" />
+		<origin xyz="0 0 0" rpy="0 0 3.14"/>
 		<parent link="base_footprint" />
 		<child link="base_link" />
@@ -292,5 +292,5 @@
 	</link>
 	<link name="head_pan_link">
-		<visual>
+		<!-- <visual>
 			<origin xyz="0 0 ${height_head_pan/2}" rpy="0 0 0"/>
 			<geometry>
@@ -300,5 +300,5 @@
 				<color rgba="0 1 0 1.0"/>
 			</material>
-		</visual>
+		</visual> -->
 		<collision>
 			<origin xyz="0 0 ${height_head_pan/2}" rpy="0 0 0"/>
@@ -309,42 +309,7 @@
 		<xacro:default_inertia mass="0.125"/>
 	</link>
-	<link name="head_tilt_link">
-		<visual>
-			<origin xyz="0 0 ${height_head_tilt/2}" rpy="0 0 0"/>
-			<geometry>
-				<box size="0.03 0.038 ${height_head_tilt}"/>
-			</geometry>
-			<material name="Green1">
-				<color rgba="0 1 0 1.0"/>
-			</material>
-		</visual>
-		<collision>
-			<origin xyz="0 0 ${height_head_tilt/2}" rpy="0 0 0"/>
-			<geometry>
-       				<box size="0.03 0.038 ${height_head_tilt}"/>
-			</geometry>
-		</collision>
-		<xacro:default_inertia mass="0.125"/>
-	</link>
-	<link name="kinect_base_link">
-		<visual>
-			<origin xyz="0 0 ${length_base/2}" rpy="0 0 0"/>
-			<geometry>
-				<box size="0.06 0.065 ${length_base}"/>
-			</geometry>
-			<material name="Green3">
-				<color rgba="0.1 0.5 0.1 1.0"/>
-			</material>
-		</visual>
-		<collision>
-			<geometry>
-       				<box size="0.06 0.065 ${length_base}"/>
-			</geometry>
-		</collision>
-		<xacro:default_inertia mass="0.125"/>
-	</link>
 	<link name="screen_link">
 		<visual>
-			<origin xyz="0.06 0 -0.11" rpy="0 -0.5 0"/>
+			<origin xyz="0.06 0 -0.11" rpy="0 0.5 3.14"/>
 			<geometry>
 				<box size="0.01 0.3 0.16"/>
@@ -355,5 +320,5 @@
 		</visual>
 		<collision>
-			<origin xyz="0.06 0 -0.11" rpy="0 -0.5 0"/>
+			<origin xyz="0.06 0 -0.11" rpy="0 0.5 3.14"/>
 			<geometry>
        				<box size="0.01 0.3 0.16"/>
@@ -371,5 +336,5 @@
  </joint>
  <joint name="base_to_wheel2" type="continuous">
-   <axis xyz="0 0 1" />
+   <axis xyz="0 0 -1" />
    <anchor xyz="0 0 0" />
    <limit effort="100" velocity="100" />
@@ -388,5 +353,5 @@
  <joint name="base_to_wheel4" type="continuous">
    <parent link="base_link"/>
-   <axis xyz="0 0 1" />
+   <axis xyz="0 0 -1" />
    <child link="wheel_4"/>
    <origin rpy="-1.5707 0 0" xyz="0 0.195 0"/>
@@ -427,18 +392,8 @@
 		<origin xyz="0 0 ${length_base}" rpy="0 0 0"/>
 	</joint>
-	<joint name="head_pan_joint" type="fixed">
+	<joint name="screen_joint" type="fixed">
 		<parent link="head_pan_link"/>
-		<child link="head_tilt_link"/>
-		<origin xyz="0 0 ${height_head_pan}" rpy="0 0 0"/>
-	</joint>
-	<joint name="kinect_base_joint" type="fixed">
-		<parent link="head_tilt_link"/>
-		<child link="kinect_base_link"/>
-		<origin xyz="0 0 ${height_head_tilt}" rpy="0 0 0"/>
-	</joint>
-	<joint name="screen_joint" type="fixed">
-		<parent link="top_torso_link"/>
 		<child link="screen_link"/>
-		<origin xyz="0 0 0.025" rpy="0 0 0"/>
+		<origin xyz="0 0 0.025" rpy="0 0 3.14"/>
 	</joint>
 </robot>

File: urdf/sensors/hokuyo.xacro (robot description, xacro)
@@ -1,8 +1,4 @@
 <?xml version="1.0"?>
 <robot name="hokuyo_sensor" xmlns:xacro="http://www.ros.org/wiki/xacro">
- <!--
- <xacro:include filename="$(find turtlebot_description)/urdf/turtlebot_gazebo.urdf.xacro"/>
- <xacro:include filename="$(find turtlebot_description)/urdf/turtlebot_properties.urdf.xacro"/>
- -->
  <xacro:macro name="hokuyo_sensor" params="parent">
      <link name="laser">
@@ -16,5 +12,5 @@
      <origin xyz="0 0 0" rpy="0 0 0"/>
      <geometry>
-       <mesh filename="package://robot_model_gazebo/meshes/sensors/hokuyo.dae"/>
+       <mesh filename="package://deliver_rb/meshes/hokuyo.dae"/>
      </geometry>
    </visual>
@@ -27,5 +23,5 @@
  <joint name="laser_joint" type="fixed">
    <axis xyz="0 0 0" />
-   <origin xyz="0.168 0 0.06" rpy="0 0 0"/>
+   <origin xyz="-0.2 0.0 0.06" rpy="0 0 3.14"/>
    <parent link="${parent}"/>
    <child link="laser"/>

File: urdf/sensors/kinect.xacro (robot description, xacro)
@@ -1,98 +1,101 @@
 <?xml version="1.0"?>
-<robot name="kinect_sensor" xmlns:xacro="http://www.ros.org/wiki/xacro">
-  <xacro:include filename="$(find robot_model_gazebo)/urdf/sensors/kinect_gazebo.xacro"/>
-  <xacro:include filename="$(find robot_model_gazebo)/urdf/sensors/kinect_properties.xacro"/>
-  <!-- Kinect driver in kinect_gazebo.xacro -->
-  <!-- Parameterised in part by the values in kinect_properties.xacro -->
-  <xacro:macro name="kinect_sensor" params="parent">
-    <joint name="camera_rgb_joint" type="fixed">
-      <!--origin xyz="${cam_px} ${cam_py} ${cam_pz}" rpy="${cam_or} ${cam_op} ${cam_oy}"/-->
-      <origin xyz="0.028 ${cam_py} 0.075" rpy="${cam_or} ${cam_op} ${cam_oy}"/>
-      <parent link="${parent}"/>
-      <child link="camera_rgb_frame" />
-    </joint>
-    <link name="camera_rgb_frame">
-      <inertial>
-        <mass value="0.001" />
-        <origin xyz="0 0 0" />
-        <inertia ixx="0.0001" ixy="0.0" ixz="0.0"
-                 iyy="0.0001" iyz="0.0"
-                 izz="0.0001" />
-      </inertial>
-    </link>
-    <joint name="camera_rgb_optical_joint" type="fixed">
-      <origin xyz="0 0 0" rpy="${-M_PI/2} 0 ${-M_PI/2}" />
-      <parent link="camera_rgb_frame" />
-      <child link="camera_rgb_optical_frame" />
-    </joint>
-    <link name="camera_rgb_optical_frame">
-      <inertial>
-        <mass value="0.001" />
-        <origin xyz="0 0 0" />
-        <inertia ixx="0.0001" ixy="0.0" ixz="0.0"
-                 iyy="0.0001" iyz="0.0"
-                 izz="0.0001" />
-      </inertial>
-    </link>
-  <joint name="camera_joint" type="fixed">
-    <origin xyz="-0.031 ${-cam_py} -0.016" rpy="0 0 0"/>
-    <parent link="camera_rgb_frame"/>
-    <child link="camera_link"/>
+<robot name="kinect" xmlns:xi="http://www.w3.org/2001/XInclude"
+    xmlns:gazebo="http://playerstage.sourceforge.net/gazebo/xmlschema/#gz"
+    xmlns:model="http://playerstage.sourceforge.net/gazebo/xmlschema/#model"
+    xmlns:sensor="http://playerstage.sourceforge.net/gazebo/xmlschema/#sensor"
+    xmlns:body="http://playerstage.sourceforge.net/gazebo/xmlschema/#body"
+    xmlns:geom="http://playerstage.sourceforge.net/gazebo/xmlschema/#geom"
+    xmlns:joint="http://playerstage.sourceforge.net/gazebo/xmlschema/#joint"
+    xmlns:controller="http://playerstage.sourceforge.net/gazebo/xmlschema/#controller"
+    xmlns:interface="http://playerstage.sourceforge.net/gazebo/xmlschema/#interface"
+    xmlns:rendering="http://playerstage.sourceforge.net/gazebo/xmlschema/#rendering"
+    xmlns:renderable="http://playerstage.sourceforge.net/gazebo/xmlschema/#renderable"
+    xmlns:physics="http://playerstage.sourceforge.net/gazebo/xmlschema/#physics"
+    xmlns:xacro="http://ros.org/wiki/xacro">
+  <!-- math constants -->
+  <xacro:property name="M_PI" value="3.1415926535897931" />
+<xacro:macro name="kinect_sensor" params="parent" >
+  <joint name="base_camera_joint" type="fixed">
+    <origin xyz="0 0 0.035" rpy="0 0 3.14" />
+    <parent link="${parent}" />
+    <child link="camera_link" />
   </joint>
-    <link name="camera_link">
+  <link name="camera_link">
+    <inertial>
+      <mass value="0.01" />
+      <origin xyz="0 0 0" />
+      <inertia ixx="0.001" ixy="0.0" ixz="0.0"
+        iyy="0.001" iyz="0.0"
+        izz="0.001" />
+    </inertial>
     <visual>
-     <!--origin xyz="0 0 0" rpy="0 0 ${M_PI/2}"/-->
-     <origin xyz="0 0 0" rpy="0 0 ${M_PI/2}"/>
+      <origin xyz=" 0 0 0 " rpy="0 0 1.57" />
       <geometry>
-       <mesh filename="package://robot_model_gazebo/meshes/sensors/kinect.dae"/>
+        <mesh filename="package://deliver_rb/meshes/kinect.dae"/>
       </geometry>
     </visual>
-	  <collision>
-      <origin xyz="0.0 0.0 0.0" rpy="0 0 0"/>
-	    <geometry>
-	      <box size="0.07271 0.27794 0.073"/>
-	    </geometry>
-	  </collision>
+    <collision>
+      <origin xyz="0.0 0.0 0.0" rpy="0 0 1.57" />
+      <geometry>
+        <box size="0.0730 .2760 0.0720"/>
+      </geometry>
+    </collision>
+  </link>
+  <joint name="camera_depth_joint" type="fixed">
+    <origin xyz="0 0.011 0" rpy="0 0 0" />
+    <parent link="camera_link" />
+    <child link="camera_depth_frame" />
+  </joint>
+  <link name="camera_depth_frame">
+    <inertial>
+      <mass value="0.01" />
+      <origin xyz="0 0 0" />
+      <inertia ixx="0.001" ixy="0.0" ixz="0.0"
+        iyy="0.001" iyz="0.0"
+        izz="0.001" />
+    </inertial>
+  </link>
+  <joint name="camera_depth_optical_joint" type="fixed">
+    <origin xyz="0 0 0" rpy="${-M_PI/2} 0 ${-M_PI/2}" />
+    <parent link="camera_depth_frame" />
+    <child link="camera_depth_optical_frame" />
+  </joint>
+  <link name="camera_depth_optical_frame">
     <inertial>
       <mass value="0.001" />
       <origin xyz="0 0 0" />
       <inertia ixx="0.0001" ixy="0.0" ixz="0.0"
-               iyy="0.0001" iyz="0.0"
-               izz="0.0001" />
+        iyy="0.0001" iyz="0.0"
+        izz="0.0001" />
     </inertial>
   </link>
-  <!-- The fixed joints & links below are usually published by static_transformers launched by the OpenNi launch
-       files. However, for Gazebo simulation we need them, so we add them here.
-       (Hence, don't publish them additionally!) -->
-	<joint name="camera_depth_joint" type="fixed">
-	  <origin xyz="0 ${2 * -cam_py} 0" rpy="0 0 0" />
-	  <parent link="camera_rgb_frame" />
-	  <child link="camera_depth_frame" />
-	</joint>
-	<link name="camera_depth_frame">
+  <joint name="camera_rgb_joint" type="fixed">
+    <origin xyz="0 -0.012 0" rpy="0 0 0" />
+    <parent link="camera_link" />
+    <child link="camera_rgb_frame" />
+  </joint>
+  <link name="camera_rgb_frame">
     <inertial>
       <mass value="0.001" />
       <origin xyz="0 0 0" />
       <inertia ixx="0.0001" ixy="0.0" ixz="0.0"
-               iyy="0.0001" iyz="0.0"
-               izz="0.0001" />
+        iyy="0.0001" iyz="0.0"
+        izz="0.0001" />
     </inertial>
-	</link>
-	<joint name="camera_depth_optical_joint" type="fixed">
-	  <origin xyz="0 0 0" rpy="${-M_PI/2} 0 ${-M_PI/2}" />
-	  <parent link="camera_depth_frame" />
-	  <child link="camera_depth_optical_frame" />
-	</joint>
-	<link name="camera_depth_optical_frame">
+  </link>
+  <joint name="camera_rgb_optical_joint" type="fixed">
+    <origin xyz="0 0 0" rpy="${-M_PI/2} 0 ${-M_PI/2}" />
+    <parent link="camera_rgb_frame" />
+    <child link="camera_rgb_optical_frame" />
+  </joint>
+  <link name="camera_rgb_optical_frame">
     <inertial>
       <mass value="0.001" />
       <origin xyz="0 0 0" />
       <inertia ixx="0.0001" ixy="0.0" ixz="0.0"
-               iyy="0.0001" iyz="0.0"
-               izz="0.0001" />
+        iyy="0.0001" iyz="0.0"
+        izz="0.0001" />
     </inertial>
-	</link>
-	<!-- Kinect sensor for simulation -->
-	<turtlebot_sim_3dsensor/>
-  </xacro:macro>
+  </link>
+</xacro:macro>
 </robot>

File: urdf/sensors/view_camera.xacro (robot description, xacro)
@@ -3,5 +3,5 @@
   <xacro:macro name="view_camera_sensor" params="parent">
   <joint name="view_camera_joint" type="continuous">
-      <origin xyz="0 0 6" rpy="0 1.570796 0"/>
+      <origin xyz="0 0 0" rpy="0 1.570796 0"/>
       <parent link="${parent}"/>
       <child link="view_camera_link" />
